File: hardware/CM5_BMW_NavBridge_0.3/Buck_Converter_5V.kicad_sch (KiCad schematic)
At the start: 17 parts, among them U1 LMR14030SQDDARQ1_C485548, U8 TPS2117DRLR_C22399676

Commit message: deleted contents of buck converter and ibus
Parts:
- removed C1: 100µ, Capacitor_SMD:CP_Elec_6.3x5.8, symbol Device:C_Polarized
- removed C2: 10µ, Capacitor_SMD:C_1206_3216Metric_Pad1.33x1.80mm_HandSolder, symbol Device:C
- removed C3, C4, C5: 0.1µ, Capacitor_SMD:C_0603_1608Metric_Pad1.08x0.95mm_HandSolder, symbol Device:C
- removed C6, C7: 47µ, Capacitor_SMD:C_1210_3225Metric_Pad1.33x2.70mm_HandSolder, symbol Device:C
- removed D1: SMCJ24A, Diode_SMD:D_SMC, symbol Device:D_Zener
- removed D2: SS54, Diode_SMD:D_SMA, symbol Device:D_Schottky
- removed F1: Fuse, Fuse:Fuseholder_Littelfuse_Nano2_154x, symbol Device:Fuse
- removed L1: 6.8uH, Inductor_SMD:L_Sunlord_MWSA1003S, symbol Device:L
- removed R1: 49.9k, Resistor_SMD:R_0603_1608Metric_Pad0.98x0.95mm_HandSolder, symbol Device:R
- removed R2: 10k, Resistor_SMD:R_0603_1608Metric_Pad0.98x0.95mm_HandSolder, symbol Device:R
- removed R3: 100k, Resistor_SMD:R_0603_1608Metric_Pad0.98x0.95mm_HandSolder, symbol Device:R
- removed R4: 17.4k, Resistor_SMD:R_0603_1608Metric_Pad0.98x0.95mm_HandSolder, symbol Device:R
- removed U1: LMR14030SQDDARQ1_C485548, JLCPCB_Misc:SOPOWERPAD-8_L4.9-W3.9-P1.27-LS6.0-BL-EP, symbol JLCPCB_Misc:LMR14030SQDDARQ1_C485548
- removed U8: TPS2117DRLR_C22399676, JLCPCB_Interface:SOT-583-8_L2.1-W1.2-P0.50-LS1.6-BL, symbol JLCPCB_Interface:TPS2117DRLR_C22399676
