File: hardware/CM5_BMW_NavBridge_0.3/IBUS.kicad_sch (KiCad schematic)
At the start: 5 parts, among them U5 ATA663254-GAQW, U6 ATmega32U4-A

Commit message: deleted contents of buck converter and ibus
Parts:
- removed C18: 10µ, Capacitor_SMD:C_1206_3216Metric_Pad1.33x1.80mm_HandSolder, symbol Device:C
- removed C19: 0.1µ, Capacitor_SMD:C_0603_1608Metric_Pad1.08x0.95mm_HandSolder, symbol Device:C
- removed R13: 10k, Resistor_SMD:R_0603_1608Metric_Pad0.98x0.95mm_HandSolder, symbol Device:R
- removed U5: ATA663254-GAQW, JLCPCB_Interface_ICs:SOIC-8_L4.9-W3.9-P1.27-LS6.0-BL, symbol JLCPCB_Interface_ICs:ATA663254-GAQW
- removed U6: ATmega32U4-A, Package_QFP:TQFP-44_10x10mm_P0.8mm, symbol MCU_Microchip_ATmega:ATmega32U4-A
Connections:
- no-connect marks 1 -> 0
