File: hardware/CM5_BMW_NavBridge_0.3/CM5_BMW_NavBridge.kicad_pcb (KiCad board)
At the start: 4 copper layers, 100 x 100 mm, 153 parts, among them CN1 10164227-1001A1RLF, CN2 10164227-1001A1RLF, CN3 X1313 Car connector, CN4 Molex to X1313 NAV connector, CN5 1-2199230-5, J1 Conn_01x04, J2 USB_A, J3 USB_C_Receptacle_USB2.0_16P, J4 Conn_01x03, J5 Conn_01x02, J7 Conn_02x03_Odd_Even, SW1 SW_nRPIBOOT, SW2 SW_DIP_x02, SW3 SW_DIP_x01, SW4 SW_RESET, SW5 SW_DIP_x01, U1 LMR14030SQDDARQ1_C485548, U10 TPS2117DRLR_C22399676, U11 PCM2912APJTR, U12 AP63203WU, U2 ADV7125KSTZ50, U3 TS5V330CDR, U4 ATA663254-GAQW, U5 ATmega32U4-A, U6 TPS2116DRL, U7 TPS2069CDBV, U8 TPS2051BDBVR, U9 TS3USB30EDGSR, Y1 Crystal_16MHz, Y2 Crystal_6MHz, Y3 ASEK-32.768KHZ-LRT

Commit message: finalized deletions and updated net deletes
Parts:
- removed C10, C12: 0.01µ, Capacitor_SMD:C_0603_1608Metric_Pad1.08x0.95mm_HandSolder
- removed C11, C13, C14, C15, C16, C9: 0.1µ, Capacitor_SMD:C_0603_1608Metric_Pad1.08x0.95mm_HandSolder
- removed C17: 10µ, Capacitor_SMD:C_1206_3216Metric_Pad1.33x1.80mm_HandSolder
- removed CN3: X1313 Car connector, Connector_PinHeader_2.54mm:PinHeader_2x09_P2.54mm_Horizontal
- removed CN4: Molex to X1313 NAV connector, Connector_Molex:Molex_Micro-Fit_3.0_43045-1200_2x06_P3.00mm_Horizontal
- removed D8: 1N4148W, Diode_SMD:D_SOD-123
- removed R10, R12, R22, R24: 10k, Resistor_SMD:R_0603_1608Metric_Pad0.98x0.95mm_HandSolder
- removed R6: 560, Resistor_SMD:R_0603_1608Metric_Pad0.98x0.95mm_HandSolder
- removed R7, R8, R9: 75, Resistor_SMD:R_0603_1608Metric_Pad0.98x0.95mm_HandSolder
- removed U2: ADV7125KSTZ50, JLCPCB_Data_Converters:LQFP-48_L7.0-W7.0-P0.50-LS9.0-BL
- removed U3: TS5V330CDR, JLCPCB_Communication_Interface_Chip_UART_485_232:SOIC-16_L9.9-W3.9-P1.27-LS6.0-BL
- removed U4: ATA663254-GAQW, JLCPCB_Interface_ICs:SOIC-8_L4.9-W3.9-P1.27-LS6.0-BL
Connections:
- U5 pad 12: MCU_LIN_EN -> MCU_IGN_SENSE
- U5 pad 20: MCU_RX -> unconnected-(U5-PD2-Pad20)
- U5 pad 21: MCU_TX -> unconnected-(U5-PD3-Pad21)
- U5 pad 40: MCU_SWITCHER_IN -> unconnected-(U5-PF1-Pad40)
- U5 pad 41: MCU_DAC_EN -> unconnected-(U5-PF0-Pad41)
Routing:
- net (no net): track 0.00 -> 468.0 mm, vias 0 -> 12
- net IBUS: track 64.2 -> 0.00 mm, vias 1 -> 0
- net NAV_AUDIO_NEG: track 58.5 -> 0.00 mm
- net NAV_AUDIO_POS: track 51.5 -> 0.00 mm
- net B_OUT: track 40.1 -> 0.00 mm, vias 1 -> 0
- net MCU_SWITCHER_IN: track 38.1 -> 0.00 mm, vias 2 -> 0
- net R_OUT: track 37.0 -> 0.00 mm, vias 1 -> 0
- net R_NAV: track 33.2 -> 0.00 mm, vias 2 -> 0
- net B_RPI: track 32.4 -> 0.00 mm, vias 2 -> 0
- net G_OUT: track 29.0 -> 0.00 mm, vias 1 -> 0
- net G_NAV: track 28.6 -> 0.00 mm, vias 2 -> 0
- net BLANK: track 26.7 -> 0.00 mm, vias 2 -> 0
- net MCU_DAC_EN: track 21.4 -> 0.00 mm, vias 2 -> 0
- net G_RPI: track 19.9 -> 0.00 mm
- net B_NAV: track 19.6 -> 0.00 mm
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