File: hardware/CM5_BMW_NavBridge_0.3/MCU_Lin.kicad_sch (KiCad schematic)
At the start: 31 parts, among them J7 Conn_02x03_Odd_Even, SW4 SW_RESET, SW5 SW_DIP_x01, U4 ATA663254-GAQW, U5 ATmega32U4-A, U6 TPS2116DRL, Y1 Crystal_16MHz

Commit message: finalized deletions and updated net deletes
Parts:
- removed C16: 0.1µ, Capacitor_SMD:C_0603_1608Metric_Pad1.08x0.95mm_HandSolder, symbol Device:C
- removed C17: 10µ, Capacitor_SMD:C_1206_3216Metric_Pad1.33x1.80mm_HandSolder, symbol Device:C
- removed D8: 1N4148W, Diode_SMD:D_SOD-123, symbol Diode:1N4148W
- removed R12: 10k, Resistor_SMD:R_0603_1608Metric_Pad0.98x0.95mm_HandSolder, symbol Device:R
- removed U4: ATA663254-GAQW, JLCPCB_Interface_ICs:SOIC-8_L4.9-W3.9-P1.27-LS6.0-BL, symbol JLCPCB_Interface_ICs:ATA663254-GAQW
Connections:
- net MCU_DAC_EN: no longer names the net of U5.41 (PF0)
- net MCU_LIN_EN renamed MCU_IGN_SENSE
- net MCU_RX: no longer names the net of U5.20 (PD2)
- net MCU_SWITCHER_IN: no longer names the net of U5.40 (PF1)
- net MCU_TX: no longer names the net of U5.21 (PD3)
- no-connect marks 13 -> 16
Other:
- note removed: "LIN"
